File: BenchBudEE.sch (KiCad schematic (older format))
At the start: 0 parts

Commit message: Thermocouple and fan
Changed lines of the file:
@@
 LIBS:contrib
 LIBS:valves
+LIBS:BenchBudEE-cache
 EELAYER 27 0
 EELAYER END
@@
 Sheet 1 8
 Title ""
-Date "27 jan 2014"
+Date "5 feb 2014"
 Rev ""
 Comp ""
@@
 $EndSheet
 $Sheet
-S 6150 1300 1600 1100
+S 6150 900  1650 1600
 U 52E653B1
 F0 "Fan" 89
 F1 "fan.sch" 89
-F2 "Power+" O R 7750 1600 60
-F3 "Power-" I R 7750 1800 60
-F4 "Tach_out" O L 6150 1750 60
-F5 "Fan_in" I L 6150 1500 60
-F6 "Tach" I R 7750 2100 60
+F2 "Power+" O R 7800 1200 60
+F3 "Power-" I R 7800 1400 60
+F4 "Tach_out" O L 6150 2200 60
+F5 "Fan_in" I L 6150 1100 60
+F6 "Tach" I R 7800 1700 60
+F7 "Current Measure" O L 6150 2050 60
+F8 "MOSI" I L 6150 1300 60
+F9 "MISO" O L 6150 1450 60
+F10 "CS_N" I L 6150 1600 60
+F11 "SCLK" I L 6150 1750 60
 $EndSheet
 $Sheet

Commit message: Power
Changed lines of the file:
@@
 LIBS:valves
 LIBS:benchBuddy
+LIBS:-12p
 LIBS:BenchBudEE-cache
 EELAYER 27 0
@@
 $Descr A4 11693 8268
 encoding utf-8
-Sheet 1 8
+Sheet 1 9
 Title ""
-Date "6 feb 2014"
+Date "7 feb 2014"
 Rev ""
 Comp ""
@@
 F1 "terminal_block.sch" 89
 $EndSheet
+$Sheet
+S 3450 1350 1750 1100
+U 52F4AA4D
+F0 "PowerAdjustmentMonitor" 89
+F1 "powerAdjustmentMonitor.sch" 89
+$EndSheet
 $EndSCHEMATC
