File: led_driver.sch (KiCad schematic (older format))
At the start: 0 parts

Commit message: LED Driver
Parts:
- added C? (x2): C, ~, symbol C
- added D?: DIODESCH, ~, symbol DIODESCH
- added L?: INDUCTOR, ~, symbol INDUCTOR
- added R?: R, ~, symbol R
- added U?: AP5726, symbol AP5726
Connections:
- net labels added: +5V, GND, LED_EN_PWM
- net labels removed: EN, FREQ
- wire segments 0 -> 17
Changed lines of the file:
@@
 LIBS:fe_v+
 LIBS:fe_v-
+LIBS:ap5726
 LIBS:BenchBudEE-cache
 EELAYER 27 0
@@
 Comment4 ""
 $EndDescr
-Text HLabel 1950 1850 0    60   Input ~ 0
-EN
-Text HLabel 1950 2550 0    60   Input ~ 0
-FREQ
-Text HLabel 7850 2100 0    60   Output ~ 0
+Text HLabel 9300 1500 2    60   Output ~ 0
 String+
-Text HLabel 7800 2750 0    60   Input ~ 0
+Text HLabel 9350 2650 2    60   Input ~ 0
 String-
+$Comp
+L AP5726 U?
+U 1 1 52F5405E
+P 3500 2400
+F 0 "U?" H 3700 1900 60  0000 C CNN
+F 1 "AP5726" H 3550 2350 60  0000 C CNN
+F 2 "" H 3500 1800 60  0000 C CNN
+F 3 "" H 3500 1800 60  0000 C CNN
+	1    3500 2400
+	1    0    0    -1
+$EndComp
+Text HLabel 1850 2450 0    60   Input ~ 0
+LED_EN_PWM
+Wire Wire Line
+	1850 2450 2850 2450
+$Comp
+L +5V #PWR?
+U 1 1 52F54222
+P 2650 1400
+F 0 "#PWR?" H 2650 1490 20  0001 C CNN
+F 1 "+5V" H 2650 1490 30  0000 C CNN
+F 2 "" H 2650 1400 60  0000 C CNN
+F 3 "" H 2650 1400 60  0000 C CNN
+	1    2650 1400
+	1    0    0    -1
+$EndComp
+$Comp
+L INDUCTOR L?
+U 1 1 52F54231
+P 3700 1500
+F 0 "L?" V 3650 1500 40  0000 C CNN
+F 1 "INDUCTOR" V 3800 1500 40  0000 C CNN
+F 2 "~" H 3700 1500 60  0000 C CNN
+F 3 "~" H 3700 1500 60  0000 C CNN
+	1    3700 1500
+	0    -1   -1   0
+$EndComp
+$Comp
+L C C?
+U 1 1 52F54240
+P 2650 1800
+F 0 "C?" H 2650 1900 40  0000 L CNN
+F 1 "C" H 2656 1715 40  0000 L CNN
+F 2 "~" H 2688 1650 30  0000 C CNN
+F 3 "~" H 2650 1800 60  0000 C CNN
+	1    2650 1800
+	1    0    0    -1
+$EndComp
+$Comp
+L C C?
+U 1 1 52F5424F
+P 8050 1950
+F 0 "C?" H 8050 2050 40  0000 L CNN
+F 1 "C" H 8056 1865 40  0000 L CNN
+F 2 "~" H 8088 1800 30  0000 C CNN
+F 3 "~" H 8050 1950 60  0000 C CNN
+	1    8050 1950
+	1    0    0    -1
+$EndComp
+$Comp
+L R R?
+U 1 1 52F5425E
+P 4800 3050
+F 0 "R?" V 4880 3050 40  0000 C CNN
+F 1 "R" V 4807 3051 40  0000 C CNN
+F 2 "~" V 4730 3050 30  0000 C CNN
+F 3 "~" H 4800 3050 30  0000 C CNN
+	1    4800 3050
+	1    0    0    -1
+$EndComp
+$Comp
+L DIODESCH D?
+U 1 1 52F5427D
+P 4850 1500
+F 0 "D?" H 4850 1600 40  0000 C CNN
+F 1 "DIODESCH" H 4850 1400 40  0000 C CNN
+F 2 "~" H 4850 1500 60  0000 C CNN
+F 3 "~" H 4850 1500 60  0000 C CNN
+	1    4850 1500
+	1    0    0    -1
+$EndComp
+$Comp
+L GND #PWR?
+U 1 1 52F5428C
+P 3550 3350
+F 0 "#PWR?" H 3550 3350 30  0001 C CNN
+F 1 "GND" H 3550 3280 30  0001 C CNN
+F 2 "" H 3550 3350 60  0000 C CNN
+F 3 "" H 3550 3350 60  0000 C CNN
+	1    3550 3350
+	1    0    0    -1
+$EndComp
+$Comp
+L GND #PWR?
+U 1 1 52F5429B
+P 2650 2150
+F 0 "#PWR?" H 2650 2150 30  0001 C CNN
+F 1 "GND" H 2650 2080 30  0001 C CNN
+F 2 "" H 2650 2150 60  0000 C CNN
+F 3 "" H 2650 2150 60  0000 C CNN
+	1    2650 2150
+	1    0    0    -1
+$EndComp
+$Comp
+L GND #PWR?
+U 1 1 52F542AA
+P 8050 2450
+F 0 "#PWR?" H 8050 2450 30  0001 C CNN
+F 1 "GND" H 8050 2380 30  0001 C CNN
+F 2 "" H 8050 2450 60  0000 C CNN
+F 3 "" H 8050 2450 60  0000 C CNN
+	1    8050 2450
+	1    0    0    -1
+$EndComp
+Wire Wire Line
+	5050 1500 9300 1500
+Wire Wire Line
+	8050 1500 8050 1750
+Connection ~ 8050 1500
+Wire Wire Line
+	8050 2450 8050 2150
+Wire Wire Line
+	3550 3100 3550 3350
+Wire Wire Line
+	4800 3300 3550 3300
+Connection ~ 3550 3300
+Wire Wire Line
+	4250 2650 9350 2650
+Wire Wire Line
+	4800 2800 4800 2650
+Connection ~ 4800 2650
+Wire Wire Line
+	4250 2450 5200 2450
+Wire Wire Line
+	5200 2450 5200 1500
+Connection ~ 5200 1500
+Wire Wire Line
+	3700 1850 4300 1850
+Wire Wire Line
+	4300 1850 4300 1500
+Wire Wire Line
+	4000 1500 4650 1500
+Connection ~ 4300 1500
+Wire Wire Line
+	2650 2000 2650 2150
+Wire Wire Line
+	2650 1400 2650 1600
+Wire Wire Line
+	3400 1500 2650 1500
+Connection ~ 2650 1500
+Wire Wire Line
+	3300 1850 3300 1500
+Connection ~ 3300 1500
 $EndSCHEMATC

Commit message: Arduino
Connections:
- net labels added: LED_STRING+, LED_STRING-
- net labels removed: String+, String-
Changed lines of the file:
@@
 LIBS:fe_v-
 LIBS:ap5726
+LIBS:arduino_pins
 LIBS:BenchBudEE-cache
 EELAYER 27 0
@@
 Sheet 6 9
 Title ""
-Date "7 feb 2014"
+Date "8 feb 2014"
 Rev ""
 Comp ""
@@
 $EndDescr
 Text HLabel 9300 1500 2    60   Output ~ 0
-String+
-Text HLabel 9350 2650 2    60   Input ~ 0
-String-
+LED_STRING+
+Text HLabel 9350 2650 2    60   Output ~ 0
+LED_STRING-
 $Comp
 L AP5726 U?
