File: thermocouple5.sch (KiCad schematic (older format))
At the start: 0 parts

Commit message: Thermocouple and fan
Parts:
- added C?: C, ~, symbol C
- added D?: ZENER, ~, symbol ZENER
- added R? (x7): R, ~, symbol R
- added U? (x4): LM324, symbol LM324
- added U? (x2): MCP3550-60-E/SN, SO8, symbol MCP3550-60-E/SN
Connections:
- net CS_N: now also U?.7 (~CS~)
- net MISO: now also U?.6 (SDO/~RDY~)
- net SCLK: now also U?.5 (SCK)
- net TC IN +: now also U?.2 (-)
- net TC IN -: now also U?.3 (+)
- new net: R?.1, R?.2, U?.1
- new net: R?.1, R?.2, U?.3 (+) (x2)
- new net: R?.2, R?.2, U?.1
- new net: R?.1, R?.2, U?.2 (-) (x2)
- new net: R?.1, U?.1, U?.2 (Vin+)
- new net: U?.1, U?.2 (Vin+), U?.3 (+)
- new net +12V: D?.2 (K), U?.11 (V-), U?.2 (-), U?.4 (V+), U?.4 (V+)
- new net -12V: U?.11 (V-), U?.11 (V-), U?.4 (V+)
- new net AGND: R?.1, U?.3 (Vin-), U?.3 (Vin-)
Other:
- note added: "16-24bit ADC"
- note added: "Analig/IC Input"
- note added: "General Temperature Sensor"
- note added: "Thermocouple Amp"
